File: ALU/ALU/_autosave-ALU.sch (KiCad schematic (older format))
At the start: 105 parts

Commit message: 25oct
Connections:
- no-connect marks 49 -> 48
Changed lines of the file:
@@
 NoConn ~ 2400 5600
 NoConn ~ 2400 5700
-NoConn ~ 4900 9800
 $Comp
 L TinyRisc_Symbol_Library:74F86 XOR41
