File: ALU/ALU/ALU.kicad_pcb (KiCad board)
At the start: 2 copper layers, 290 x 194 mm, 105 parts

Commit message: 27oct
Finished v1.0 of ALU, PC and GP RF.
Updated documentation to match.
Parts:
- removed C3, C37, C4, C5: 100nF, Capacitors_THT:C_Axial_L5.1mm_D3.1mm_P7.50mm_Horizontal
- removed DECODEAND0: 74F8, Housings_DIP:DIP-14_W7.62mm
- removed DECODENOT0: 74F04, Housings_DIP:DIP-14_W7.62mm
- removed DECODEOR1, DECODEOR2, DECODEROR0, DECODEROR1: 74F32, Housings_DIP:DIP-14_W7.62mm
- added DEC1: 74F138, Package_DIP:DIP-16_W7.62mm, F.Cu at (116.0, 163.0)
- added NAND41: 74F00, Package_DIP:DIP-14_W7.62mm, F.Cu at (115.0, 205.0)
- 5V/GND1: footprint Connectors_JST:JST_XH_B02B-XH-A_02x2.50mm_Straight -> Connector_JST:JST_XH_B2B-XH-AM_1x02_P2.50mm_Vertical
- ADD4.0, ADD4.1, ADD4.2, ADD4.3, MUXCout1: footprint Housings_DIP:DIP-16_W7.62mm -> Package_DIP:DIP-16_W7.62mm
- ADD_GATE0, ADD_GATE1, AND_GATE1, COMP1, FlagsAdd0, FlagsLeft1, FlagsLogical1, FlagsRight1, NAND_GATE0, OR_GATE1, SL_GATE0, SR_GATE0, XOR_GATE0: footprint Housings_DIP:DIP-20_W7.62mm -> Package_DIP:DIP-20_W7.62mm
- ALU_COMM1, FLAGS_OUT1: footprint Kicad Libraries:09185067904 -> Kicad libraries:6pinIDC
- ALU_OUT1, OP1, OP2: footprint Kicad Libraries:16pinIDC -> Kicad libraries:16pinIDC
- AND0, AND1, NAND0, NAND1, OR0, OR1, OverflowXOR1, XOR0, XOR1, XOR2, XOR3, XOR4, XOR41: footprint Housings_DIP:DIP-14_W7.62mm -> Package_DIP:DIP-14_W7.62mm
- C1, C10, C11, C12, C13, C14, C15, C16, C17, C18, C19, C2, C20, C21, C22, C23, C24, C25, C26, C27, C28, C29, C30, C31, C32, C33, C34, C35, C36, C6, C7, C8, C9: footprint Capacitors_THT:C_Axial_L5.1mm_D3.1mm_P7.50mm_Horizontal -> Capacitor_THT:C_Axial_L5.1mm_D3.1mm_P7.50mm_Horizontal
- CPOWER1: footprint Capacitors_THT:CP_Radial_D8.0mm_P2.50mm -> Capacitor_THT:CP_Radial_D8.0mm_P2.50mm
- H1, H2, H3, H4, H5, H6, H7, H8: footprint Mounting_Holes:MountingHole_3.5mm_Pad_Via -> MountingHole:MountingHole_3.5mm_Pad_Via
- PD10, PD11, PD12, PD13, PD14, PD15, PD8, PD9, PDB10, PDB11, PDB12, PDB13, PDB14, PDB15, PDB8, PDB9: footprint Resistors_THT:R_Axial_DIN0204_L3.6mm_D1.6mm_P7.62mm_Horizontal -> Resistor_THT:R_Axial_DIN0204_L3.6mm_D1.6mm_P7.62mm_Horizontal
- moved H1 265.8 mm to (325.0, 35.0)
- moved H3 255.0 mm to (325.0, 225.0)
- moved H5 235.9 mm to (95.0, 35.0)
- moved H2 225.1 mm to (95.0, 225.0)
- moved C31 215.7 mm to (118.0, 142.0), turned to 180 degrees
- moved FlagsLogical1 205.8 mm to (118.0, 136.0), turned to 180 degrees
- moved SL_GATE0 193.8 mm to (176.0, 220.0), turned to 90 degrees
- moved NAND0 187.1 mm to (88.0, 59.0)
- moved H4 186.7 mm to (85.0, 35.0)
- moved NAND1 186.3 mm to (88.0, 87.0)
- moved NAND_GATE0 184.9 mm to (110.0, 68.0)
- moved C15 182.5 mm to (322.0, 56.0)
- moved C19 181.8 mm to (171.0, 220.0)
- moved C8 181.0 mm to (295.0, 73.0), turned to 0 degrees
- moved H6 180.7 mm to (85.0, 225.0)
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Connections:
- ADD4.2 pad 10: /S11 -> ADD_CX
- ADD4.2 pad 9: ADD_CX -> Net-(ADD4.2-Pad9)
- ADD4.3 pad 7: ADD_CX -> Net-(ADD4.2-Pad9)
- ADD_GATE1 pad 5: /S11 -> ADD_CX
- OverflowXOR1 pad 6: AXORB -> ~LOG_EN
Routing:
- net GNDREF: track 0.00 -> 1794.1 mm
- net +5V: track 0.00 -> 1487.8 mm, vias 0 -> 1
- net /O0: track 0.00 -> 612.3 mm, vias 0 -> 4
- net Logical_N: track 0.00 -> 608.2 mm, vias 0 -> 2
- net SL_COUT: track 0.00 -> 593.0 mm, vias 0 -> 2
- net /O1: track 0.00 -> 577.9 mm, vias 0 -> 2
- net /O5: track 0.00 -> 576.1 mm, vias 0 -> 2
- net /O2: track 0.00 -> 572.3 mm, vias 0 -> 2
- net /A5: track 0.00 -> 571.2 mm, vias 0 -> 2
- net /O6: track 0.00 -> 562.7 mm, vias 0 -> 3
- net /A4: track 0.00 -> 561.7 mm, vias 0 -> 2
- net /O4: track 0.00 -> 559.4 mm
- net /O3: track 0.00 -> 557.4 mm, vias 0 -> 3
- net SL_N: track 0.00 -> 553.6 mm, vias 0 -> 4
- net SR_COUT: track 0.00 -> 529.8 mm, vias 0 -> 2
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- removed copper zone on B.Cu, net GNDREF
Other:
- board size 290 x 194 mm -> 260 x 200 mm
- net class Power added: clearance 0.3, trace_width 0.4, via_dia 0.8, via_drill 0.4
- board text added: "5V"
- board text added: "ADD: 1100 SUB: 1101 LEFT SHIFT: 0001 LEFT ROTATE: 0000 RIGHT SHIFT: 0011 RIGHT ROTATE: 0010"
- board text added: "ALU COMM + FLAGS In"
- board text added: "ALU COMMAND CODES"
- board text added: "ALU OUPUT"
- board text added: "AND array"
- board text added: "AND: 100X OR: 010X XOR: 101X NAND:011X"
- board text added: "Adder and Subtractor"
- board text added: "FLAGS OUT"
- board text added: "FLAGS logic"
- board text added: "GND"
- board text added: "NAND ARRAY"
- board text added: "OR ARRAY"
- board text added: "OR Array"
- board text added: "Operand 1"
- board text added: "Operand 2"
- board text added: "Shifter Unit (L/R)"
- board text added: "TinyRISC ALU (rev. 1.0) Creator: Luc Boulesteix"
