File: ALU/ALU/ALU.sch (KiCad schematic (older format))
At the start: 105 parts

Commit message: 27oct
Finished v1.0 of ALU, PC and GP RF.
Updated documentation to match.
Parts:
- removed C3, C37, C4, C5: 100nF, Capacitors_THT:C_Axial_L5.1mm_D3.1mm_P7.50mm_Horizontal, symbol Device:C
- removed DECODEAND0: 74F8, Housings_DIP:DIP-14_W7.62mm, symbol TinyRisc_Symbol_Library:74F8
- removed DECODENOT0: 74F04, Housings_DIP:DIP-14_W7.62mm, symbol TinyRisc_Symbol_Library:74F04
- removed DECODEOR1, DECODEOR2, DECODEROR0, DECODEROR1: 74F32, Housings_DIP:DIP-14_W7.62mm, symbol TinyRisc_Symbol_Library:74F32
- added DEC1: 74F138, Package_DIP:DIP-16_W7.62mm, symbol TinyRisc_Symbol_Library:74F138
- added NAND41: 74F00, Package_DIP:DIP-14_W7.62mm, symbol TinyRisc_Symbol_Library:74F00
- 5V/GND1: footprint Connectors_JST:JST_XH_B02B-XH-A_02x2.50mm_Straight -> Connector_JST:JST_XH_B2B-XH-AM_1x02_P2.50mm_Vertical
- ADD4.0, ADD4.1, ADD4.2, ADD4.3, MUXCout1: footprint Housings_DIP:DIP-16_W7.62mm -> Package_DIP:DIP-16_W7.62mm
- ADD_GATE0, ADD_GATE1, AND_GATE1, COMP1, FlagsAdd0, FlagsLeft1, FlagsLogical1, FlagsRight1, NAND_GATE0, OR_GATE1, SL_GATE0, SR_GATE0, XOR_GATE0: footprint Housings_DIP:DIP-20_W7.62mm -> Package_DIP:DIP-20_W7.62mm
- ALU_COMM1, FLAGS_OUT1: footprint Kicad Libraries:09185067904 -> Kicad libraries:6pinIDC
- ALU_OUT1, OP1, OP2: footprint Kicad Libraries:16pinIDC -> Kicad libraries:16pinIDC
- AND0, AND1, NAND0, NAND1, OR0, OR1, OverflowXOR1, XOR0, XOR1, XOR2, XOR3, XOR4, XOR41: footprint Housings_DIP:DIP-14_W7.62mm -> Package_DIP:DIP-14_W7.62mm
- C1, C10, C11, C12, C13, C14, C15, C16, C17, C18, C19, C2, C20, C21, C22, C23, C24, C25, C26, C27, C28, C29, C30, C31, C32, C33, C34, C35, C36, C6, C7, C8, C9: footprint Capacitors_THT:C_Axial_L5.1mm_D3.1mm_P7.50mm_Horizontal -> Capacitor_THT:C_Axial_L5.1mm_D3.1mm_P7.50mm_Horizontal
- CPOWER1: footprint Capacitors_THT:CP_Radial_D8.0mm_P2.50mm -> Capacitor_THT:CP_Radial_D8.0mm_P2.50mm
- H1, H2, H3, H4, H5, H6, H7, H8: footprint Mounting_Holes:MountingHole_3.5mm_Pad_Via -> MountingHole:MountingHole_3.5mm_Pad_Via
- PD10, PD11, PD12, PD13, PD14, PD15, PD8, PD9, PDB10, PDB11, PDB12, PDB13, PDB14, PDB15, PDB8, PDB9: footprint Resistors_THT:R_Axial_DIN0204_L3.6mm_D1.6mm_P7.62mm_Horizontal -> Resistor_THT:R_Axial_DIN0204_L3.6mm_D1.6mm_P7.62mm_Horizontal
Connections:
- net AXORB is gone; now on net ~LOG_EN: OverflowXOR1.6 (O1)
- net S11 is gone; now on net ADD_CX: ADD4.2.10 (S3), ADD_GATE1.5 (A3)
- net +5V: now also DEC1.16 (VCC), DEC1.6 (G1), NAND41.14 (VCC)
- net A: now also DEC1.1 (A)
- net ADD_CX: no longer ADD4.2.9 (Cout), ADD4.3.7 (Cin)
- net B: now also DEC1.2 (B)
- net C: now also DEC1.3 (C)
- net GNDREF: now also DEC1.4 (~G2A), DEC1.5 (~G2B), DEC1.8 (GND), NAND41.7 (GND)
- net Z: now also NAND41.3 (O0)
- net ~ADDER_EN: now also DEC1.12 (Y3)
- net ~AND_EN: now also DEC1.14 (Y1)
- net ~LEFT_EN: now also DEC1.15 (Y0)
- net ~NAND_EN: now also DEC1.9 (Y6)
- net ~OR_EN: now also DEC1.13 (Y2)
- net ~RIGHT_EN: now also DEC1.11 (Y4)
- net ~XOR_EN: now also DEC1.10 (Y5)
- net ~Z: now also NAND41.1 (A0), NAND41.2 (B0)
- new net: ADD4.2.9 (Cout), ADD4.3.7 (Cin)
- no-connect marks 49 -> 42
Other:
- note added: "Subtituting NOT for NAND"
- note removed: "!A+B"
- note removed: "!C+!D"
- note removed: "!C+D"
- note removed: "(A.B)+!C"
- note removed: "(A.B)+C\n"
- note removed: "A.B"
- note removed: "C+!D"
- note removed: "C+D"
