File: Program Counter/V1.0/Program Counter.sch (KiCad schematic (older format))
At the start: 42 parts, among them J1 PC_OUT, J2 PC_OFFS, J3 Control, J4 Clock

Commit message: oct22
Parts:
- removed ADD1, ADD2, ADD3, ADD4: 74F283, symbol TinyRisc~Symbol~Library:74F283
- removed MUX1A1, MUX1B1, MUX2A1, MUX2B1, MUX3A1, MUX4A1: 74F257, symbol TinyRisc~Symbol~Library:74F257
- removed R1, R2: 1K, symbol Device:R
- removed R12, R13, R15: 10k, symbol Device:R
- removed R16, R3: 10K, symbol Device:R
- added ADD4.1, ADD4.2, ADD4.3, ADD4.4: 74F283, Housings_DIP:DIP-16_W7.62mm, symbol TinyRisc~Symbol~Library:74F283
- added C_BOARD1: 10uF, Capacitors_THT:CP_Radial_D8.0mm_P2.50mm, symbol Device:CP1_Small
- added H1, H2, H3, H4: MountingHole, Mounting_Holes:MountingHole_3.5mm_Pad_Via, symbol Mechanical:MountingHole
- added H5, H6, H7, H8: MountingHole_Pad, Mounting_Holes:MountingHole_3.5mm_Pad_Via, symbol Mechanical:MountingHole_Pad
- added J5: POWER/GND, Connectors_JST:JST_NV_B02P-NV_2x5.00mm_Vertical, symbol Connector:Conn_01x02_Male
- added MUXA1, MUXA2, MUXA3, MUXA4, MUXB1, MUXB2: 74F257, Housings_DIP:DIP-16_W7.62mm, symbol TinyRisc~Symbol~Library:74F257
- C1, C10, C11, C12, C13, C2, C3, C4, C5, C6, C7, C8, C9: footprint (none) -> Capacitors_THT:C_Axial_L5.1mm_D3.1mm_P7.50mm_Horizontal
- J1, J2: footprint (none) -> Connectors_JST:JST_XH_B16B-XH-A_16x2.50mm_Straight
- J3: footprint (none) -> Connectors_JST:JST_XH_B04B-XH-A_04x2.50mm_Straight
- J4: footprint (none) -> Connectors:1pin
- POT1: footprint (none) -> Potentiometers:Potentiometer_Trimmer_ACP_CA14h5_Vertical_Px5.0mm_Py10.0mm
- R10, R14, R4, R5, R6: footprint (none) -> Resistors_THT:R_Axial_DIN0204_L3.6mm_D1.6mm_P7.62mm_Horizontal
- REG8.1, REG8.2: footprint (none) -> Housings_DIP:DIP-24_W7.62mm
Connections:
- net labels added: GND
- net labels removed: n7, s11, s12, ~OE_ABS
- wire segments 356 -> 418
- no-connect marks 0 -> 1

Commit message: 25oct
Parts:
- J1, J2: footprint Connectors_JST:JST_XH_B16B-XH-A_16x2.50mm_Straight -> Kicad Libraries:16pinIDC
Changed lines of the file:
@@
 F 0 "J1" H 5950 3717 50  0000 C CNN
 F 1 "PC_OUT" H 5950 3626 50  0000 C CNN
-F 2 "Connectors_JST:JST_XH_B16B-XH-A_16x2.50mm_Straight" H 5900 3200 50  0001 C CNN
+F 2 "Kicad Libraries:16pinIDC" H 5900 3200 50  0001 C CNN
 F 3 "~" H 5900 3200 50  0001 C CNN
 	1    5900 3200
@@
 F 0 "J2" H 7850 6117 50  0000 C CNN
 F 1 "PC_OFFS" H 7850 6026 50  0000 C CNN
-F 2 "Connectors_JST:JST_XH_B16B-XH-A_16x2.50mm_Straight" H 7800 5600 50  0001 C CNN
+F 2 "Kicad Libraries:16pinIDC" H 7800 5600 50  0001 C CNN
 F 3 "~" H 7800 5600 50  0001 C CNN
 	1    7800 5600
@@
 Wire Wire Line
 	6050 1300 5800 1300
-Wire Bus Line
-	6450 2800 6450 3800
-Wire Bus Line
-	6950 1550 6950 4950
-Wire Bus Line
-	8350 5200 8350 6400
-Wire Bus Line
-	7050 4950 7050 6400
-Wire Bus Line
-	5600 2800 5600 3800
-Wire Bus Line
-	8650 750  8650 6000
-Wire Bus Line
-	850  950  850  7750
-Wire Bus Line
-	10850 1250 10850 6050
-Wire Bus Line
-	1150 1000 1150 7700
-Wire Bus Line
-	9050 1450 9050 6400
-Wire Bus Line
-	2400 1200 2400 6950
-Wire Bus Line
-	3450 1200 3450 3800
-Wire Bus Line
-	5200 1200 5200 3800
 Connection ~ 6050 1550
 Connection ~ 5800 1300
@@
 	1    0    0    -1
 $EndComp
+Wire Bus Line
+	6450 2800 6450 3800
+Wire Bus Line
+	6950 1550 6950 4950
+Wire Bus Line
+	8350 5200 8350 6400
+Wire Bus Line
+	7050 4950 7050 6400
+Wire Bus Line
+	5600 2800 5600 3800
+Wire Bus Line
+	8650 750  8650 6000
+Wire Bus Line
+	850  950  850  7750
+Wire Bus Line
+	10850 1250 10850 6050
+Wire Bus Line
+	1150 1000 1150 7700
+Wire Bus Line
+	9050 1450 9050 6400
+Wire Bus Line
+	2400 1200 2400 6950
+Wire Bus Line
+	3450 1200 3450 3800
+Wire Bus Line
+	5200 1200 5200 3800
 $EndSCHEMATC

Commit message: 25oct
Parts:
- removed J3: Control, Connectors_JST:JST_XH_B04B-XH-A_04x2.50mm_Straight, symbol Connector:Conn_01x04_Male
- added J3: Control, Kicad Libraries:6pinIDC, symbol Connector:Conn_01x06_Male
Connections:
- no-connect marks 1 -> 3
Changed lines of the file:
@@
 CLK
-$Comp
-L Connector:Conn_01x04_Male J3
-U 1 1 6303158B
-P 5750 5900
-F 0 "J3" H 5722 5782 50  0000 R CNN
-F 1 "Control" H 5722 5873 50  0000 R CNN
-F 2 "Connectors_JST:JST_XH_B04B-XH-A_04x2.50mm_Straight" H 5750 5900 50  0001 C CNN
-F 3 "~" H 5750 5900 50  0001 C CNN
-	1    5750 5900
-	-1   0    0    1
-$EndComp
 $Comp
 L Connector:Conn_01x01_Male J4
@@
 $EndComp
 Wire Wire Line
-	4500 5700 5550 5700
-Wire Wire Line
 	5350 5850 5350 5800
 Wire Wire Line
-	5350 5800 5550 5800
-Wire Wire Line
 	5350 6000 5350 5900
 Wire Wire Line
-	5350 5900 5550 5900
-Wire Wire Line
 	5450 6150 5450 6000
-Wire Wire Line
-	5450 6000 5550 6000
 Wire Wire Line
 	5050 6150 5450 6150
@@
 	1    0    0    -1
 $EndComp
+$Comp
+L Connector:Conn_01x06_Male J3
+U 1 1 617B196B
+P 5950 5800
+F 0 "J3" H 5922 5682 50  0000 R CNN
+F 1 "Control" H 5922 5773 50  0000 R CNN
+F 2 "Kicad Libraries:6pinIDC" H 5950 5800 50  0001 C CNN
+F 3 "~" H 5950 5800 50  0001 C CNN
+	1    5950 5800
+	-1   0    0    1
+$EndComp
+Wire Wire Line
+	5450 6000 5750 6000
+Wire Wire Line
+	5350 5900 5750 5900
+Wire Wire Line
+	5350 5800 5750 5800
+Wire Wire Line
+	4500 5700 5750 5700
+NoConn ~ 5750 5500
+NoConn ~ 5750 5600
 Wire Bus Line
 	6450 2800 6450 3800

Commit message: 27oct
Finished v1.0 of ALU, PC and GP RF.
Updated documentation to match.
Parts:
- J1, J2: footprint Kicad Libraries:16pinIDC -> Kicad libraries:16pinIDC
- J4: footprint Connectors:1pin -> Connector_Pin:Pin_D1.0mm_L10.0mm
- J5: footprint Connectors_JST:JST_NV_B02P-NV_2x5.00mm_Vertical -> Connector_JST:JST_PH_B2B-PH-K_1x02_P2.00mm_Vertical
- J6: renamed from J3; footprint Kicad Libraries:6pinIDC -> Kicad libraries:6pinIDC
Changed lines of the file:
@@
 F 0 "J1" H 5950 3717 50  0000 C CNN
 F 1 "PC_OUT" H 5950 3626 50  0000 C CNN
-F 2 "Kicad Libraries:16pinIDC" H 5900 3200 50  0001 C CNN
+F 2 "Kicad libraries:16pinIDC" H 5900 3200 50  0001 C CNN
 F 3 "~" H 5900 3200 50  0001 C CNN
 	1    5900 3200
@@
 F 0 "J2" H 7850 6117 50  0000 C CNN
 F 1 "PC_OFFS" H 7850 6026 50  0000 C CNN
-F 2 "Kicad Libraries:16pinIDC" H 7800 5600 50  0001 C CNN
+F 2 "Kicad libraries:16pinIDC" H 7800 5600 50  0001 C CNN
 F 3 "~" H 7800 5600 50  0001 C CNN
 	1    7800 5600
@@
 F 0 "J4" H 5722 6232 50  0000 R CNN
 F 1 "Clock" H 5722 6323 50  0000 R CNN
-F 2 "Connectors:1pin" H 5750 6300 50  0001 C CNN
+F 2 "Connector_Pin:Pin_D1.0mm_L10.0mm" H 5750 6300 50  0001 C CNN
 F 3 "~" H 5750 6300 50  0001 C CNN
 	1    5750 6300
@@
 F 0 "J5" V 5762 744 50  0000 L CNN
 F 1 "POWER/GND" V 5650 450 50  0000 L CNN
-F 2 "Connectors_JST:JST_NV_B02P-NV_2x5.00mm_Vertical" H 5700 700 50  0001 C CNN
+F 2 "Connector_JST:JST_PH_B2B-PH-K_1x02_P2.00mm_Vertical" H 5700 700 50  0001 C CNN
 F 3 "~" H 5700 700 50  0001 C CNN
 	1    5700 700
@@
 $EndComp
 $Comp
-L Connector:Conn_01x06_Male J3
+L Connector:Conn_01x06_Male J6
 U 1 1 617B196B
 P 5950 5800
-F 0 "J3" H 5922 5682 50  0000 R CNN
+F 0 "J6" H 5922 5682 50  0000 R CNN
 F 1 "Control" H 5922 5773 50  0000 R CNN
-F 2 "Kicad Libraries:6pinIDC" H 5950 5800 50  0001 C CNN
+F 2 "Kicad libraries:6pinIDC" H 5950 5800 50  0001 C CNN
 F 3 "~" H 5950 5800 50  0001 C CNN
 	1    5950 5800
